File: modulo_sensor/modulo_sensor.kicad_sch (KiCad schematic)
At the start: 33 parts, among them J1 Conn_01x08_Pin, U1 74HC14DR2G

Commit message: feat: Placa doble faz
Placa 120x30mm doble faz
Parts:
- D1, D2, D3, D4, D5, D6: footprint LED_THT:LED_D3.0mm -> LED_SMD:LED_1206_3216Metric_Pad1.42x1.75mm_HandSolder
Connections:
- net GND: now also J1.8 (Pin_8); no longer J1.4 (Pin_4)
- net Led_Sensor1: now also J1.5 (Pin_5); no longer J1.7 (Pin_7)
- net Led_Sensor2: now also J1.4 (Pin_4); no longer J1.6 (Pin_6)
- net Led_Sensor3: now also J1.3 (Pin_3); no longer J1.5 (Pin_5)
- net Led_Sensor4: now also J1.2 (Pin_2), U1.2 (1Y); no longer J1.3 (Pin_3), U1.6 (3Y)
- net Led_Sensor5: now also J1.6 (Pin_6); no longer J1.2 (Pin_2)
- net Led_Sensor6: now also J1.7 (Pin_7), U1.6 (3Y); no longer J1.1 (Pin_1), U1.2 (1Y)
- net Sensor4: now also U1.1 (1A); no longer U1.5 (3A)
- net Sensor6: now also U1.5 (3A); no longer U1.1 (1A)
- net vcc: now also J1.1 (Pin_1); no longer J1.8 (Pin_8)
