File: modulo_seguidor/modulo_seguidor.kicad_pcb (KiCad board)
At the start: 12 copper layers, 100 x 50 mm, 12 parts, among them J1 Battery, J4 Motor Izquierdo, J5 Motor Derecho, J6 puerto sensores, SW1 SW_Push, U1 LM7806_TO220

Commit message: refactor: Muevo los pines al lado del arduino nano
Reorganizo las conexiones pero nos ahorramos los cables de los sensores
Parts:
- J6: footprint Connector_PinHeader_2.54mm:PinHeader_1x08_P2.54mm_Horizontal -> Connector_PinHeader_2.54mm:PinHeader_1x08_P2.54mm_Vertical
- moved J6 19.3 mm to (129.5, 58.4), turned to -90 degrees
- moved C1 10.2 mm to (94.0, 91.4)
- moved R2 10.2 mm to (132.1, 88.9)
- moved U1 10.2 mm to (106.7, 88.9)
- moved A2 10.2 mm to (95.2, 71.1)
- moved C2 10.2 mm to (114.3, 86.4)
- moved D1 10.2 mm to (124.5, 88.9)
- moved J1 10.2 mm to (81.3, 86.4), turned to -90 degrees
- moved J4 10.2 mm to (86.4, 71.1)
- moved J5 10.2 mm to (86.4, 76.2)
- moved R1 7.78 mm to (78.7, 53.3), turned to -90 degrees
- moved SW1 2.11 mm to (93.5, 58.3)
Connections:
- A2 pad D10: /PWM_IZQ -> /Boton_encendido
- A2 pad D2: /Boton_encendido -> /Sensor6
- A2 pad D3: /Sensor6 -> /Sensor5
- A2 pad D4: /Sensor5 -> /Sensor4
- A2 pad D5: /Sensor4 -> /Sensor3
- A2 pad D6: /Sensor3 -> /Sensor2
- A2 pad D7: /Sensor2 -> /Sensor1
- A2 pad D8: /Sensor1 -> /PWM_DER
- A2 pad D9: /PWM_DER -> /PWM_IZQ
- J6 pad 1: /Sensor6 -> VCC
- J6 pad 2: /Sensor5 -> GND
- J6 pad 3: /Sensor4 -> /Sensor6
- J6 pad 4: /Sensor3 -> /Sensor5
- J6 pad 5: /Sensor2 -> /Sensor4
- J6 pad 6: /Sensor1 -> /Sensor3
- J6 pad 7: VCC -> /Sensor2
- J6 pad 8: GND -> /Sensor1
Routing:
- net /Sensor1: track 58.0 -> 5.08 mm
- net /Sensor2: track 54.1 -> 5.08 mm
- net /Sensor3: track 50.1 -> 5.08 mm
- net /Sensor4: track 46.1 -> 5.08 mm
- net /Sensor5: track 42.3 -> 5.08 mm
- net GND: track 174.9 -> 139.1 mm
- net /Sensor6: track 38.1 -> 5.08 mm
- net /Boton_encendido: track 44.6 -> 35.1 mm
- net VCC: track 99.2 -> 104.2 mm
- net /PWM_IZQ: track 25.4 -> 27.9 mm
- net /PWM_DER: track 33.0 -> 35.6 mm
- net +5V: track 60.9 -> 59.4 mm
