File: modulo_seguidor/modulo_seguidor.kicad_sch (KiCad schematic)
At the start: 12 parts, among them J1 Battery, J4 Motor Izquierdo, J5 Motor Derecho, J6 puerto sensores, SW1 SW_Push, U1 LM7806_TO220

Commit message: refactor: Muevo los pines al lado del arduino nano
Reorganizo las conexiones pero nos ahorramos los cables de los sensores
Parts:
- J6: footprint Connector_PinHeader_2.54mm:PinHeader_1x08_P2.54mm_Horizontal -> Connector_PinHeader_2.54mm:PinHeader_1x08_P2.54mm_Vertical
Connections:
- net Boton_encendido: now also A2.D10; no longer A2.D2 (D2_INT0)
- net GND: now also J6.2 (Pin_2); no longer J6.8 (Pin_8)
- net PWM_DER: now also A2.D8; no longer A2.D9
- net PWM_IZQ: now also A2.D9; no longer A2.D10
- net Sensor1: now also A2.D7, J6.8 (Pin_8); no longer A2.D8, J6.6 (Pin_6)
- net Sensor2: now also A2.D6, J6.7 (Pin_7); no longer A2.D7, J6.5 (Pin_5)
- net Sensor3: now also A2.D5, J6.6 (Pin_6); no longer A2.D6, J6.4 (Pin_4)
- net Sensor4: now also A2.D4, J6.5 (Pin_5); no longer A2.D5, J6.3 (Pin_3)
- net Sensor5: now also A2.D3 (D3_INT1), J6.4 (Pin_4); no longer A2.D4, J6.2 (Pin_2)
- net Sensor6: now also A2.D2 (D2_INT0), J6.3 (Pin_3); no longer A2.D3 (D3_INT1), J6.1 (Pin_1)
- net VCC: now also J6.1 (Pin_1); no longer J6.7 (Pin_7)
Other:
- moved on the sheet: J6
